File: pcb/sciencecamp_logger.kicad_pcb (KiCad board)
At the start: 2 copper layers, 97 x 46 mm, 33 parts, among them J1 1-Wire, J2 HC-SR04, J3 OLED, J4 Micro_SD_Card_Det, SW1 OFF/ON, SW2 action, U1 74LVC125, U2 AMS1117-3.3

Commit message: ADD: url
Other:
- board text added: "Data↔D7"
- board text added: "SCL←A5"
- board text added: "SDA↔A4"
- board text added: "echo→D2"
- board text added: "https://logger.educatweb.de/2019"
- board text added: "trigger←D6"
- board text added: "→D2"
- board text removed: "Data"
- board text removed: "SCL"
- board text removed: "SDA"
- board text removed: "echo"
- board text removed: "trigger"
Changed lines of the file:
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@@
   (general
     (thickness 1.6)
-    (drawings 27)
+    (drawings 29)
     (tracks 340)
     (zones 0)
@@
   (page A4)
   (layers
-    (0 F.Cu signal)
-    (31 B.Cu signal)
+    (0 F.Cu signal hide)
+    (31 B.Cu signal hide)
     (32 B.Adhes user)
     (33 F.Adhes user)
@@
     (descr "Arduino Nano, http://www.mouser.com/pdfdocs/Gravitech_Arduino_Nano3_0.pdf")
     (tags "Arduino Nano")
-    (fp_text reference A1 (at 7.62 -5.08 90) (layer F.SilkS)
+    (fp_text reference A1 (at 7.62 -5.08 90) (layer F.Fab)
       (effects (font (size 1 1) (thickness 0.15)))
     )
@@
     )
   )
-  (gr_text trigger (at 122.25 97.75) (layer B.SilkS)
+  (gr_text https://logger.educatweb.de/2019 (at 136.5 114.5) (layer F.SilkS)
+    (effects (font (size 1 1) (thickness 0.15)))
+  )
+  (gr_text →D2 (at 149.75 111.25) (layer F.SilkS)
+    (effects (font (size 1 1) (thickness 0.15)))
+  )
+  (gr_text trigger←D6 (at 123.75 97.75) (layer B.SilkS)
     (effects (font (size 1 1) (thickness 0.15)) (justify mirror))
   )
-  (gr_text echo (at 121.5 100.5) (layer B.SilkS)
+  (gr_text echo→D2 (at 123 100.5) (layer B.SilkS)
     (effects (font (size 1 1) (thickness 0.15)) (justify mirror))
   )
@@
     (effects (font (size 1 1) (thickness 0.15)) (justify mirror))
   )
-  (gr_text SDA (at 156.75 102.75) (layer F.SilkS)
+  (gr_text SDA↔A4 (at 155.25 102.75) (layer F.SilkS)
     (effects (font (size 1 1) (thickness 0.15)))
   )
-  (gr_text SCL (at 156.75 100.25) (layer F.SilkS)
+  (gr_text SCL←A5 (at 155.25 100) (layer F.SilkS)
     (effects (font (size 1 1) (thickness 0.15)))
   )
@@
     (effects (font (size 1 1) (thickness 0.15)))
   )
-  (gr_text Data (at 121 84.5) (layer F.SilkS)
+  (gr_text Data↔D7 (at 122.5 84.5) (layer F.SilkS)
     (effects (font (size 1 1) (thickness 0.15)))
   )

Commit message: UPD: more THT
Parts:
- R12, R13: footprint Resistor_SMD:R_0603_1608Metric_Pad1.05x0.95mm_HandSolder -> Resistor_THT:R_Axial_DIN0309_L9.0mm_D3.2mm_P12.70mm_Horizontal
- moved R13 25.9 mm to (154.4, 78.3)
- moved R12 23.2 mm to (160.1, 78.3)
Routing:
- net /SDA: track 36.4 -> 50.2 mm
- net +5V: track 144.1 -> 155.5 mm
- net /SCL: track 32.4 -> 42.8 mm
- net GND: track 11.8 -> 13.7 mm, vias 43 -> 49
